File: vm1-controller/kicad/v01/vm1-controller/20231027_vm-1_prototyp/20231027_vm-1_prototyp.kicad_pcb (KiCad board)
At the start: 2 copper layers, 225 x 100 mm, 80 parts, among them J2 Conn_01x08_Pin, SW1 SW_SPST, SW10 SW_SPST, SW11 SW_SPST, SW12 SW_SPST, SW13 SW_SPST, SW14 SW_SPST, SW15 SW_SPST, SW16 SW_SPST, SW17 SW_SPST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

Commit message: updated README.md
Parts:
- R3, R4: value 0402WGF1002TCE -> 0402WGF1002TCE 10k
